Commit message: add ellipse wheel

File: urdf/carrier.urdf.xacro (robot description, xacro)
@@ -13,4 +13,7 @@
 	<inertia  ixx="${m*(r*r/4+l*l/12)}" ixy = "0" ixz = "0" iyy="${m*(r*r/4+l*l/12)}" iyz = "0" izz="${m*r*r/2}" />
 </macro>
+<macro name="ellipse_inertia" params="m short long l">
+	<inertia  ixx="${m*(short*short)/4}" ixy = "0" ixz = "0" iyy="${m*(short*short+long*long)/4}" iyz = "0" izz="${m*(long*long)/4}" />
+</macro>
 <!-- Main Body-base -->
 <property name="base_x_size" value="0.20" />
@@ -22,4 +25,9 @@
 <property name="child_body_l" value="0.15" />
 <property name="child_body_mass" value="1.30" />
+<!-- carrier robot wheel -->
+<property name="carrier_wheel_long" value="0.1" />
+<property name="carrier_wheel_short" value="0.05" />
+<property name="carrier_wheel_l" value="0.02" />
+<property name="carrier_wheel_mass" value="0.1" />
 <!-- child robot wheel -->
 <property name="child_wheel_r" value="0.075" />
@@ -53,4 +61,40 @@
    <mu2>0.2</mu2>
 </gazebo>
+<!-- ==========Carrier's left side wheel definition========== -->
+<!-- Left side wheel of carrier robot -->
+<link name="carrier_robot_wheel_L_link">
+	<inertial>
+		<mass value="${carrier_wheel_mass}" />
+		<origin xyz="0 0 0" />
+		<ellipse_inertia m="${carrier_wheel_mass}" short="${carrier_wheel_short}" long="${carrier_wheel_long}" l="${carrier_wheel_l}" />
+	</inertial>
+	<visual>
+		<origin xyz="0 0 0" rpy="0 0 0" />
+		<geometry>
+			<mesh filename="package://carrier_robot/stl/ellipse_sample.STL" />
+		</geometry>
+		<material name="Black" />
+	</visual>
+	<collision>
+		<origin xyz="0 0 0" rpy="0 0 0 " />
+		<geometry>
+			<mesh filename="package://carrier_robot/stl/ellipse_sample.STL" />
+		</geometry>
+	</collision>
+</link>
+<gazebo reference="carrier_robot_wheel_L_link">
+	<material>Gazebo/Black</material>
+	<turnGravityOff>false</turnGravityOff>
+	<mu1>0.5</mu1>
+   <mu2>0.5</mu2>
+</gazebo>
+<!-- Joint between base_link and carrier_robot_wheel_L_link -->
+<joint name="carrier_base_wheel_L_joint" type="continuous">
+	<parent link="base_link" />
+	<child link="carrier_robot_wheel_L_link"/>
+	<origin rpy="0 0 0" xyz="${(-1)*(base_x_size/2-0.05)} ${base_y_size/2+carrier_wheel_l/2} 0" />
+	<axis xyz="0 1 0" />
+</joint>
+<!--${base_y_size/2+0.01+carrier_wheel_l/2}-->
 <!-- Body of child robot-->
 <link name="child_robot_base_link">
@@ -190,5 +234,5 @@
 <gazebo>
 	<plugin name="gazebo_ros_control" filename="libgazebo_ros_control.so">
-		<robotNamespace>my_robo</robotNamespace>
+		<robotNamespace>carrier</robotNamespace>
 	</plugin>
 </gazebo>

Commit message: add many

File: urdf/carrier.urdf.xacro (robot description, xacro)
@@ -61,5 +61,50 @@
    <mu2>0.2</mu2>
 </gazebo>
-<!-- ==========Carrier's left side wheel definition========== -->
+<!-- ==========Carrier's wheels definition========== -->
+<!-- Right side wheel of carrier robot -->
+<link name="carrier_robot_wheel_R_link">
+	<inertial>
+		<mass value="${carrier_wheel_mass}" />
+		<origin xyz="0 0 0" />
+		<ellipse_inertia m="${carrier_wheel_mass}" short="${carrier_wheel_short}" long="${carrier_wheel_long}" l="${carrier_wheel_l}" />
+	</inertial>
+	<visual>
+		<origin xyz="0 0 0" rpy="0 0 0" />
+		<geometry>
+			<mesh filename="package://carrier_robot/stl/ellipse_sample.STL" />
+		</geometry>
+		<material name="Black" />
+	</visual>
+	<collision>
+		<origin xyz="0 0 0" rpy="0 0 0 " />
+		<geometry>
+			<mesh filename="package://carrier_robot/stl/ellipse_sample.STL" />
+		</geometry>
+	</collision>
+</link>
+<gazebo reference="carrier_robot_wheel_R_link">
+	<material>Gazebo/Black</material>
+	<turnGravityOff>false</turnGravityOff>
+	<mu1>0.5</mu1>
+   <mu2>0.5</mu2>
+</gazebo>
+<!-- Joint between base_link and carrier_robot_wheel_R_link -->
+<joint name="carrier_base_wheel_R_joint" type="continuous">
+	<parent link="base_link" />
+	<child link="carrier_robot_wheel_R_link"/>
+	<origin rpy="0 0 0" xyz="${(-1)*(base_x_size/2-0.05)} ${(-1)*(base_y_size/2+0.02+carrier_wheel_l/2)} 0" />
+	<axis xyz="0 1 0" />
+</joint>
+<!-- Transmission of carrier_base_wheel_R_joint -->
+<transmission name="carrier_base_wheel_R_joint_trans">
+	<type>transmission_interface/SimpleTransmission</type>
+	<joint name="carrier_base_wheel_R_joint">
+		<hardwareInterface>hardware_interface/VelocityJointInterface</hardwareInterface>
+	</joint>
+	<actuator name="carrier_base_wheel_R_joint_motor">
+		<hardwareInterface>hardware_interface/VelocityJointInterface</hardwareInterface>
+		<mechanicalReduction>1</mechanicalReduction>
+	</actuator>
+</transmission>
 <!-- Left side wheel of carrier robot -->
 <link name="carrier_robot_wheel_L_link">
@@ -89,12 +134,11 @@
    <mu2>0.5</mu2>
 </gazebo>
-<!-- Joint between base_link and carrier_robot_wheel_L_link -->
-<joint name="carrier_base_wheel_L_joint" type="continuous">
-	<parent link="base_link" />
+<!-- Joint between carrier_robot_wheel_R_link and carrier_robot_wheel_L_link -->
+<joint name="carrier_wheel_R-L_joint" type="fixed">
+	<parent link="carrier_robot_wheel_R_link" />
 	<child link="carrier_robot_wheel_L_link"/>
-	<origin rpy="0 0 0" xyz="${(-1)*(base_x_size/2-0.05)} ${base_y_size/2+carrier_wheel_l/2} 0" />
-	<axis xyz="0 1 0" />
-</joint>
-<!--${base_y_size/2+0.01+carrier_wheel_l/2}-->
+	<origin rpy="0 0 0" xyz="0 ${base_y_size+0.02+carrier_wheel_l} 0" />
+	<!--<origin rpy="0 0 0" xyz="${(-1)*(base_x_size/2-0.05)} ${base_y_size/2+carrier_wheel_l/2} 0" /> -->
+</joint>
 <!-- Body of child robot-->
 <link name="child_robot_base_link">
@@ -169,8 +213,8 @@
 	<type>transmission_interface/SimpleTransmission</type>
 	<joint name="child_base_wheel_R_joint">
-		<hardwareInterface>hardware_interface/EffortJointInterface</hardwareInterface>
+		<hardwareInterface>hardware_interface/VelocityJointInterface</hardwareInterface>
 	</joint>
 	<actuator name="child_base_wheel_R_joint_motor">
-		<hardwareInterface>hardware_interface/EffortJointInterface</hardwareInterface>
+		<hardwareInterface>hardware_interface/VelocityJointInterface</hardwareInterface>
 		<mechanicalReduction>1</mechanicalReduction>
 	</actuator>
@@ -216,8 +260,8 @@
 	<type>transmission_interface/SimpleTransmission</type>
 	<joint name="child_base_wheel_L_joint">
-		<hardwareInterface>hardware_interface/EffortJointInterface</hardwareInterface>
+		<hardwareInterface>hardware_interface/VelocityJointInterface</hardwareInterface>
 	</joint>
 	<actuator name="child_base_wheel_L_joint_motor">
-		<hardwareInterface>hardware_interface/EffortJointInterface</hardwareInterface>
+		<hardwareInterface>hardware_interface/VelocityJointInterface</hardwareInterface>
 		<mechanicalReduction>1</mechanicalReduction>
 	</actuator>
